File: modelos/poncho_grande/principal.sch (KiCad schematic (older format))
At the start: 10 parts, among them P1 CONN_6, P10 CONN_4, P2 CONN_4, P3 CONN_10, P4 CONN_9, P5 CONN_7, P6 CONN_7, P7 CONN_5, P8 CONN_5, P9 CONN_6

Commit message: * Agregados las asociaciones con módulos desde el esquemático.
Parts:
- removed P3: CONN_10, symbol CONN_10
- removed P4: CONN_9, symbol CONN_9
- removed P5, P6: CONN_7, symbol CONN_7
- added K1, K2: CONN_3, Connect:bornier3, symbol CONN_3
- added P11, P5, P6: CONN_4, Connect:bornier4, symbol CONN_4
- added P12, P3, P4: CONN_5, Connect:bornier5, symbol CONN_5
- P1, P9: footprint (none) -> Connect:bornier6
- P10: footprint (none) -> Connect:bornier4
- P2, P7, P8: footprint (none) -> Connect:bornier5
Changed lines of the file:
@@
 LIBS:conn
 LIBS:modelos_ponchos
-EELAYER 24 0
+LIBS:poncho_grande-cache
+EELAYER 25 0
 EELAYER END
 $Descr A4 11693 8268
@@
 F 0 "P1" V 2100 1900 60  0000 C CNN
 F 1 "CONN_6" V 2200 1900 60  0000 C CNN
-F 2 "" H 2150 1900 60  0000 C CNN
+F 2 "Connect:bornier6" H 2400 1500 60  0000 C CNN
 F 3 "" H 2150 1900 60  0000 C CNN
 	1    2150 1900
@@
 F 0 "P2" V 7900 4000 50  0000 C CNN
 F 1 "CONN_4" V 8000 4000 50  0000 C CNN
-F 2 "" H 7950 4000 60  0000 C CNN
+F 2 "Connect:bornier5" H 8100 3650 60  0000 C CNN
 F 3 "" H 7950 4000 60  0000 C CNN
 	1    7950 4000
@@
 U 1 1 560BF658
 P 7350 3800
+AR Path="/560BF658" Ref="#PWR04"  Part="1"
+AR Path="/560A0C1A/560BF658" Ref="#PWR04"  Part="1"
 F 0 "#PWR04" H 7350 3760 30  0001 C CNN
 F 1 "+3.3V" H 7350 3910 30  0000 C CNN
@@
 F 0 "P8" V 7850 2800 50  0000 C CNN
 F 1 "CONN_5" V 7950 2800 50  0000 C CNN
-F 2 "" H 7900 2800 60  0000 C CNN
+F 2 "Connect:bornier5" H 7900 2800 60  0001 C CNN
 F 3 "" H 7900 2800 60  0000 C CNN
 	1    7900 2800
@@
 U 1 1 560A36D6
 P 7200 2450
+AR Path="/560A36D6" Ref="#PWR07"  Part="1"
+AR Path="/560A0C1A/560A36D6" Ref="#PWR07"  Part="1"
 F 0 "#PWR07" H 7200 2410 30  0001 C CNN
 F 1 "+3.3V" H 7200 2560 30  0000 C CNN
@@
 Text HLabel 4450 1400 0    60   BiDi ~ 0
 COL2
-$Comp
-L CONN_10 P3
-U 1 1 560AC3FE
-P 4950 1450
-F 0 "P3" V 4900 1450 60  0000 C CNN
-F 1 "CONN_10" V 5000 1450 60  0000 C CNN
-F 2 "" H 4950 1450 60  0000 C CNN
-F 3 "" H 4950 1450 60  0000 C CNN
-	1    4950 1450
-	1    0    0    -1
-$EndComp
 Wire Wire Line
 	4600 1200 4450 1200
@@
 F 0 "P9" V 7900 5300 60  0000 C CNN
 F 1 "CONN_6" V 8000 5300 60  0000 C CNN
-F 2 "" H 7950 5300 60  0000 C CNN
+F 2 "Connect:bornier6" H 7950 5300 60  0001 C CNN
 F 3 "" H 7950 5300 60  0000 C CNN
 	1    7950 5300
@@
 Wire Wire Line
 	7600 5250 7450 5250
-$Comp
-L CONN_9 P4
-U 1 1 560AC711
-P 5000 3300
-F 0 "P4" V 4950 3300 60  0000 C CNN
-F 1 "CONN_9" V 5050 3300 60  0000 C CNN
-F 2 "" H 5000 3300 60  0000 C CNN
-F 3 "" H 5000 3300 60  0000 C CNN
-	1    5000 3300
-	1    0    0    -1
-$EndComp
-$Comp
-L CONN_7 P5
-U 1 1 560AC725
-P 5000 5200
-F 0 "P5" V 4970 5200 60  0000 C CNN
-F 1 "CONN_7" V 5070 5200 60  0000 C CNN
-F 2 "" H 5000 5200 60  0000 C CNN
-F 3 "" H 5000 5200 60  0000 C CNN
-	1    5000 5200
-	1    0    0    -1
-$EndComp
-$Comp
-L CONN_7 P6
-U 1 1 560AC739
-P 5000 6450
-F 0 "P6" V 4970 6450 60  0000 C CNN
-F 1 "CONN_7" V 5070 6450 60  0000 C CNN
-F 2 "" H 5000 6450 60  0000 C CNN
-F 3 "" H 5000 6450 60  0000 C CNN
-	1    5000 6450
-	1    0    0    -1
-$EndComp
 Wire Wire Line
 	4650 3100 4400 3100
@@
 U 1 1 560AD02C
 P 7200 1050
+AR Path="/560AD02C" Ref="#PWR010"  Part="1"
+AR Path="/560A0C1A/560AD02C" Ref="#PWR010"  Part="1"
 F 0 "#PWR010" H 7200 1010 30  0001 C CNN
 F 1 "+3.3V" H 7200 1160 30  0000 C CNN
@@
 $EndComp
 $Comp
-L +5P #PWR25
+L +5P #PWR011
 U 1 1 560AD040
 P 7550 4950
-F 0 "#PWR25" H 7550 5080 20  0001 C CNN
+F 0 "#PWR011" H 7550 5080 20  0001 C CNN
 F 1 "+5P" H 7550 5050 30  0000 C CNN
 F 2 "" H 7550 4950 60  0000 C CNN
@@
 $EndComp
 $Comp
-L +5P #PWR9
+L +5P #PWR012
 U 1 1 560AD068
 P 4500 4800
-F 0 "#PWR9" H 4500 4930 20  0001 C CNN
+F 0 "#PWR012" H 4500 4930 20  0001 C CNN
 F 1 "+5P" H 4500 4900 30  0000 C CNN
 F 2 "" H 4500 4800 60  0000 C CNN
@@
 $EndComp
 $Comp
-L +5P #PWR11
+L +5P #PWR013
 U 1 1 560AD07C
 P 4500 6100
-F 0 "#PWR11" H 4500 6230 20  0001 C CNN
+F 0 "#PWR013" H 4500 6230 20  0001 C CNN
 F 1 "+5P" H 4500 6200 30  0000 C CNN
 F 2 "" H 4500 6100 60  0000 C CNN
@@
 U 1 1 560ADA52
 P 4300 900
-F 0 "#PWR011" H 4300 860 30  0001 C CNN
+AR Path="/560ADA52" Ref="#PWR011"  Part="1"
+AR Path="/560A0C1A/560ADA52" Ref="#PWR014"  Part="1"
+F 0 "#PWR014" H 4300 860 30  0001 C CNN
 F 1 "+3.3V" H 4300 1010 30  0000 C CNN
 F 2 "" H 4300 900 60  0000 C CNN
@@
 $EndComp
 $Comp
-L +5V #PWR012
+L +5V #PWR015
 U 1 1 560ADA66
 P 7400 1050
-F 0 "#PWR012" H 7400 1140 20  0001 C CNN
+F 0 "#PWR015" H 7400 1140 20  0001 C CNN
 F 1 "+5V" H 7400 1140 30  0000 C CNN
 F 2 "" H 7400 1050 60  0000 C CNN
@@
 $EndComp
 $Comp
-L +5P #PWR13
+L +5P #PWR016
 U 1 1 560ADA8E
 P 4550 2800
-F 0 "#PWR13" H 4550 2930 20  0001 C CNN
+F 0 "#PWR016" H 4550 2930 20  0001 C CNN
 F 1 "+5P" H 4550 2900 30  0000 C CNN
 F 2 "" H 4550 2800 60  0000 C CNN
@@
 $EndComp
 $Comp
-L +3.3VP #PWR013
+L +3.3VP #PWR017
 U 1 1 560ADAA2
 P 4350 2800
-F 0 "#PWR013" H 4400 2830 20  0001 C CNN
+F 0 "#PWR017" H 4400 2830 20  0001 C CNN
 F 1 "+3.3VP" H 4350 2890 30  0000 C CNN
 F 2 "" H 4350 2800 60  0000 C CNN
@@
 $EndComp
 $Comp
-L +3.3VP #PWR014
+L +3.3VP #PWR018
 U 1 1 560ADAB6
 P 4300 4800
-F 0 "#PWR014" H 4350 4830 20  0001 C CNN
+F 0 "#PWR018" H 4350 4830 20  0001 C CNN
 F 1 "+3.3VP" H 4300 4890 30  0000 C CNN
 F 2 "" H 4300 4800 60  0000 C CNN
@@
 U 1 1 560AE144
 P 1600 1650
-F 0 "#PWR015" H 1600 1610 30  0001 C CNN
+AR Path="/560AE144" Ref="#PWR015"  Part="1"
+AR Path="/560A0C1A/560AE144" Ref="#PWR019"  Part="1"
+F 0 "#PWR019" H 1600 1610 30  0001 C CNN
 F 1 "+3.3V" H 1600 1760 30  0000 C CNN
 F 2 "" H 1600 1650 60  0000 C CNN
@@
 	4300 1100 4300 900
 $Comp
-L +3.3VP #PWR016
+L +3.3VP #PWR020
 U 1 1 560AE1D9
 P 7350 4950
-F 0 "#PWR016" H 7400 4980 20  0001 C CNN
+F 0 "#PWR020" H 7400 4980 20  0001 C CNN
 F 1 "+3.3VP" H 7350 5040 30  0000 C CNN
 F 2 "" H 7350 4950 60  0000 C CNN
@@
 F 0 "P7" V 7850 1350 50  0000 C CNN
 F 1 "CONN_5" V 7950 1350 50  0000 C CNN
-F 2 "" H 7900 1350 60  0000 C CNN
+F 2 "Connect:bornier5" H 7900 1350 60  0001 C CNN
 F 3 "" H 7900 1350 60  0000 C CNN
 	1    7900 1350
@@
 	4500 6150 4500 6100
 $Comp
-L GND #PWR017
+L GND #PWR021
 U 1 1 560AE608
 P 4500 2000
-F 0 "#PWR017" H 4500 2000 30  0001 C CNN
+F 0 "#PWR021" H 4500 2000 30  0001 C CNN
 F 1 "GND" H 4500 1930 30  0001 C CNN
 F 2 "" H 4500 2000 60  0000 C CNN
@@
 $EndComp
 $Comp
-L GND #PWR018
+L GND #PWR022
 U 1 1 560AE61C
 P 4550 3800
-F 0 "#PWR018" H 4550 3800 30  0001 C CNN
+F 0 "#PWR022" H 4550 3800 30  0001 C CNN
 F 1 "GND" H 4550 3730 30  0001 C CNN
 F 2 "" H 4550 3800 60  0000 C CNN
@@
 $EndComp
 $Comp
-L GND #PWR019
+L GND #PWR023
 U 1 1 560AE630
 P 4500 5600
-F 0 "#PWR019" H 4500 5600 30  0001 C CNN
+F 0 "#PWR023" H 4500 5600 30  0001 C CNN
 F 1 "GND" H 4500 5530 30  0001 C CNN
 F 2 "" H 4500 5600 60  0000 C CNN
@@
 $EndComp
 $Comp
-L GND #PWR020
+L GND #PWR024
 U 1 1 560AE644
 P 4500 6850
-F 0 "#PWR020" H 4500 6850 30  0001 C CNN
+F 0 "#PWR024" H 4500 6850 30  0001 C CNN
 F 1 "GND" H 4500 6780 30  0001 C CNN
 F 2 "" H 4500 6850 60  0000 C CNN
@@
 $EndComp
 $Comp
-L GND #PWR021
+L GND #PWR025
 U 1 1 560AE658
 P 7450 1650
-F 0 "#PWR021" H 7450 1650 30  0001 C CNN
+F 0 "#PWR025" H 7450 1650 30  0001 C CNN
 F 1 "GND" H 7450 1580 30  0001 C CNN
 F 2 "" H 7450 1650 60  0000 C CNN
@@
 $EndComp
 $Comp
-L GND #PWR022
+L GND #PWR026
 U 1 1 560AE66C
 P 7550 5650
-F 0 "#PWR022" H 7550 5650 30  0001 C CNN
+F 0 "#PWR026" H 7550 5650 30  0001 C CNN
 F 1 "GND" H 7550 5580 30  0001 C CNN
 F 2 "" H 7550 5650 60  0000 C CNN
@@
 F 0 "P10" V 2150 1050 50  0000 C CNN
 F 1 "CONN_4" V 2250 1050 50  0000 C CNN
-F 2 "" H 2200 1050 60  0000 C CNN
+F 2 "Connect:bornier4" H 2500 750 60  0000 C CNN
 F 3 "" H 2200 1050 60  0000 C CNN
 	1    2200 1050
@@
 Wire Wire Line
 	1850 1100 1600 1100
+$Comp
+L CONN_4 P6
+U 1 1 560A4F90
+P 5000 5050
+F 0 "P6" V 4950 5050 50  0000 C CNN
+F 1 "CONN_4" V 5050 5050 50  0000 C CNN
+F 2 "Connect:bornier4" H 5000 5050 60  0001 C CNN
+F 3 "" H 5000 5050 60  0000 C CNN
+	1    5000 5050
+	1    0    0    -1
+$EndComp
+$Comp
+L CONN_3 K1
+U 1 1 560A4FA4
+P 5000 5400
+F 0 "K1" V 4950 5400 50  0000 C CNN
+F 1 "CONN_3" V 5050 5400 40  0000 C CNN
+F 2 "Connect:bornier3" H 5000 5400 60  0001 C CNN
+F 3 "" H 5000 5400 60  0000 C CNN
+	1    5000 5400
+	1    0    0    -1
+$EndComp
+$Comp
+L CONN_4 P11
+U 1 1 560A4FB8
+P 5000 6300
+F 0 "P11" V 4950 6300 50  0000 C CNN
+F 1 "CONN_4" V 5050 6300 50  0000 C CNN
+F 2 "Connect:bornier4" H 5000 6300 60  0001 C CNN
+F 3 "" H 5000 6300 60  0000 C CNN
+	1    5000 6300
+	1    0    0    -1
+$EndComp
+$Comp
+L CONN_3 K2
+U 1 1 560A4FCC
+P 5000 6650
+F 0 "K2" V 4950 6650 50  0000 C CNN
+F 1 "CONN_3" V 5050 6650 40  0000 C CNN
+F 2 "Connect:bornier3" H 5000 6650 60  0001 C CNN
+F 3 "" H 5000 6650 60  0000 C CNN
+	1    5000 6650
+	1    0    0    -1
+$EndComp
+$Comp
+L CONN_4 P5
+U 1 1 560A4FE0
+P 5000 3550
+F 0 "P5" V 4950 3550 50  0000 C CNN
+F 1 "CONN_4" V 5050 3550 50  0000 C CNN
+F 2 "Connect:bornier4" H 5350 3250 60  0000 C CNN
+F 3 "" H 5000 3550 60  0000 C CNN
+	1    5000 3550
+	1    0    0    -1
+$EndComp
+$Comp
+L CONN_5 P12
+U 1 1 560A4FF4
+P 5050 3100
+F 0 "P12" V 5000 3100 50  0000 C CNN
+F 1 "CONN_5" V 5100 3100 50  0000 C CNN
+F 2 "Connect:bornier5" H 5050 3100 60  0001 C CNN
+F 3 "" H 5050 3100 60  0000 C CNN
+	1    5050 3100
+	1    0    0    -1
+$EndComp
+$Comp
+L CONN_5 P3
+U 1 1 560A5008
+P 5000 1200
+F 0 "P3" V 4950 1200 50  0000 C CNN
+F 1 "CONN_5" V 5050 1200 50  0000 C CNN
+F 2 "Connect:bornier5" H 5500 1000 60  0000 C CNN
+F 3 "" H 5000 1200 60  0000 C CNN
+	1    5000 1200
+	1    0    0    -1
+$EndComp
+$Comp
+L CONN_5 P4
+U 1 1 560A501C
+P 5000 1700
+F 0 "P4" V 4950 1700 50  0000 C CNN
+F 1 "CONN_5" V 5050 1700 50  0000 C CNN
+F 2 "Connect:bornier5" H 5000 1700 60  0001 C CNN
+F 3 "" H 5000 1700 60  0000 C CNN
+	1    5000 1700
+	1    0    0    -1
+$EndComp
 $EndSCHEMATC

Commit message: * Modificaciones en el esquemático.
Parts:
- P3, P4: footprint Connect:bornier5 -> (none)
- renumbered P8 to P10, P2 to P11, P9 to P12, P10 to P2, P12 to P5, P5 to P6, P6 to P7, P11 to P8, P7 to P9

Commit message: * Mejoras y emprolijamiento en el esquemático y el PCB.
Parts:
- removed P10, P9: CONN_5, Connect:bornier5, symbol CONN_5
- added P12, P13: CONN_5, mod:bornier5, symbol CONN_5
- P1: footprint Connect:bornier6 -> mod:bornier6
- P10: renamed from K2; footprint Connect:bornier3 -> mod:bornier3
- P11: value CONN_4 -> CONN_5; footprint Connect:bornier5 -> mod:bornier5
- P14: renamed from P12; footprint Connect:bornier6 -> mod:bornier6
- P2, P6, P7: footprint Connect:bornier4 -> mod:bornier4
- P3, P4: footprint (none) -> mod:bornier5
- P5: footprint Connect:bornier5 -> mod:bornier5
- P8: renamed from K1; footprint Connect:bornier3 -> mod:bornier3
- P9: renamed from P8; footprint Connect:bornier4 -> mod:bornier4
Connections:
- net labels added: +5VP
- net labels removed: +5P

Commit message: * Cambios en el esquemático. Ejemplo de Poncho simple con área para prototipado.
Parts:
- removed P1, P14: CONN_6, mod:bornier6, symbol CONN_6
- removed P10, P8: CONN_3, mod:bornier3, symbol CONN_3
- removed P11, P12, P13, P3, P4, P5: CONN_5, mod:bornier5, symbol CONN_5
- removed P2, P6, P7, P9: CONN_4, mod:bornier4, symbol CONN_4
- added P1, P3, P4, P6, P8, P9: CONN_02X20, Pin_Headers:Pin_Header_Straight_2x20, symbol CONN_02X20
- added P10, P11: CONN_01X20, Pin_Headers:Pin_Header_Straight_1x20, symbol CONN_01X20
- added P12, P13: CONN_01X06, mod:bornier6, symbol CONN_01X06
- added P14, P15, P16, P17: CONN_02X12, Pin_Headers:Pin_Header_Straight_2x12, symbol CONN_02X12
- added P18, P19, P20, P21: CONN_01X12, Pin_Headers:Pin_Header_Straight_1x12, symbol CONN_01X12
- added P2, P7: CONN_01X20, Pin_Headers:Pin_Header_Straight_2x12, symbol CONN_02X12
- added P5: CONN_01X40, Pin_Headers:Pin_Header_Straight_1x19, symbol CONN_01X19
Connections:
- net labels added: +3.3VADC, SCL
- net labels removed: SDL
- wire segments 98 -> 366
- no-connect marks 9 -> 43

Commit message: * Actualizado el modelo de Poncho Grande. Ya terminado de rutear.
Parts:
- P5: value CONN_01X40 -> CONN_01X19
Changed lines of the file:
@@
 EESchema Schematic File Version 2
-LIBS:modelos_ponchos
-LIBS:misc
-LIBS:conn
+LIBS:Poncho_Esqueleto
+LIBS:Misc_Poncho_Grande
 LIBS:poncho_grande-cache
 EELAYER 25 0
@@
 P 7300 5800
 F 0 "P5" V 7300 6850 50  0000 C CNN
-F 1 "CONN_01X40" V 7300 4500 50  0001 C CNN
+F 1 "CONN_01X19" V 7300 4500 50  0001 C CNN
 F 2 "Pin_Headers:Pin_Header_Straight_1x19" H 7300 5800 60  0001 C CNN
 F 3 "" H 7300 5800 60  0000 C CNN
