File: Poncho EDU CIAA Amp Audio/Amp Potencia.sch (KiCad schematic (older format))
At the start: 7 parts, among them P1 CONN_01X02, U2 LM386

Commit message: v2
Connections:
- net GNDA: no longer U2.4 (Gnd)
- new net GND: U2.4 (Gnd)
Other:
- moved on the sheet: C7, C8, C9, P1, R9, RV2, U2
