File: Poncho EDU CIAA Amp Audio/Poncho EDU CIAA Amp Audio.sch (KiCad schematic (older format))
At the start: 0 parts

Commit message: v2
Parts:
- added C1: 100 uF, footprints:Kemet_ESH106M050AC3AA, symbol CP
- added C2: 22 uF, footprints:Kemet_ESH106M050AC3AA, symbol CP
- added C3: 0,022 uF, Capacitors_SMD:C_1206_HandSoldering, symbol C
- added C4: 1 uF, Capacitors_SMD:C_1206_HandSoldering, symbol C
- added C5: 100pF, Capacitors_SMD:C_1206_HandSoldering, symbol C
- added C6, C7: 10 uF, footprints:Kemet_ESH106M050AC3AA, symbol CP
- added C8: 0,047 uF, Capacitors_SMD:C_1206_HandSoldering, symbol C
- added C9: 270 uF, footprints:C_Kemet_ESY277M063AL3AA, symbol CP
- added F1, F2, F3: FIDUCIAL, ej2cese:Fiducial_1mm, symbol FIDUCIAL
- added J1: JACK_2P, footprints:Conector_mini_Plug, symbol JACK_2P
- added P1: CONN_01X02, Connect:bornier2, symbol CONN_01X02
- added R1, R2, R8: 4,7k, footprints:R_1206_HandSoldering, symbol R
- added R10: 0, footprints:R_1206_HandSoldering, symbol R
- added R3, R7: 47k, footprints:R_1206_HandSoldering, symbol R
- added R4: 560, footprints:R_1206_HandSoldering, symbol R
- added R5: 1k, footprints:R_1206_HandSoldering, symbol R
- added R6: 15k, footprints:R_1206_HandSoldering, symbol R
- added R9: 10, footprints:R_1206_HandSoldering, symbol R
- added RV1: 20k, footprints:POT_20K_0.25W_Bourns_3310C, symbol POT
- added RV2: 10 k, footprints:POT_20K_0.25W_Bourns_3310C, symbol POT
- added U1: LM741, footprints:LM741_Texas_Instruments, symbol LM741
- added U2: LM386, footprints:LM741_Texas_Instruments, symbol LM386
- added XA1: Conn_Poncho2P_2x_20x2, footprints:Conn_Poncho_Derecha, symbol Conn_Poncho2P_2x_20x2
Connections:
- new net: C5.2, R4.1, R7.2, U1.2 (-)
- new net: R5.1, U1.3 (+)
- new net: C5.1, C6.1, R7.1, U1.6
- new net: J1.1, J1.2, RV1.1
- new net: C3.1, RV1.2
- new net: C3.2, C4.1, R6.2
- new net: C4.2, R3.1, R5.2
- new net: C1.1, R1.2, R2.1, R3.2
- new net: C2.1, R4.2
- new net: C6.2, R8.2
- new net: C7.1, U2.1
- new net: RV2.2, U2.3 (+)
- new net: C8.1, C9.1, U2.5
- new net: C7.2, U2.8
- new net: C8.2, R9.1
- new net: C9.2, P1.1 (P1)
- new net +3.3V: R1.1, U1.7 (V+), XA1.1 (+3.3V)
- new net +5V: U2.6 (V+), XA1.2 (+5V)
- new net ADC: R8.1, XA1.13 (ADC1)
- new net DAC: RV2.1, XA1.15 (DAC)
- new net GND: R10.2, U1.4 (V-), U2.4 (Gnd), XA1.20 (GND), XA1.22 (GND), XA1.24 (GND), XA1.26 (GND), XA1.28 (GND), XA1.30 (GND), XA1.32 (GND), XA1.38 (GND), XA1.4 (GND), XA1.40 (GND)
- new net GNDA: C1.2, C2.2, J1.3, P1.2 (P2), R10.1, R2.2, R6.1, R9.2, RV1.3, RV2.3, U2.2 (-), XA1.10 (GNDA), XA1.12 (GNDA), XA1.14 (GNDA), XA1.16 (GNDA), XA1.18 (GNDA), XA1.7 (GNDA), XA1.8 (GNDA)
- no-connect marks 0 -> 21
Other:
- note added: "Consumo en Reposo: 4mA.\nPotencia de Salida: 275 mW (resistencia de 8 Ohms)."
- note added: "Distorsión (THD): 0.2%"
- note added: "Ganancia: de 20 hasta 200 dB"
