File: Poncho EDU CIAA Amp Audio/Poncho EDU CIAA Amp Audio.kicad_pcb (KiCad board)
At the start: 2 copper layers, 40.6 x 69.8 mm, 28 parts, among them J1 JACK_2P, P1 CONN_01X02, U1 LM741, U2 LM386

Commit message: v2
Parts:
- added F3: FIDUCIAL, ej2cese:Fiducial_1mm, F.Cu at (190.0, 76.2)
- added G101: Logo_OSHWA, footprints:Logo_OSHWA, F.Cu at (183.9, 136.4)
- added R10: 0, footprints:R_1206_HandSoldering, F.Cu at (180.0, 130.7)
- C2: value 0,022 uF -> 22 uF
- C3: value 1 uF -> 0,022 uF
- C4: value 22 uF -> 1 uF
- J1: footprint footprints:Jack_Plug_1_4_Switchcraft_Inc_RA49C12A -> footprints:Conector_mini_Plug
- R4: value 15k -> 560
- R6: value 560 -> 15k
- RV2: footprint footprints:Potentiometer_Bourns-51AAD -> footprints:POT_20K_0.25W_Bourns_3310C
- U2: footprint footprints:Texas_Instrument_LM386 -> footprints:LM741_Texas_Instruments
- moved G*** 54.9 mm to (172.3, 82.3)
- moved R6 47.9 mm to (162.1, 123.4), turned to 0 degrees
- moved C4 45.7 mm to (161.0, 128.3), turned to 0 degrees
- moved U1 41.5 mm to (177.4, 122.7), turned to 90 degrees
- moved R5 40.6 mm to (173.9, 126.0)
- moved R7 33.9 mm to (173.9, 109.2), turned to 0 degrees
- moved C5 33.6 mm to (173.9, 112.1), turned to 0 degrees
- moved C9 27.1 mm to (162.6, 83.2)
- moved C1 24.9 mm to (175.0, 140.1), turned to 180 degrees
- moved J1 21.1 mm to (154.4, 136.1), turned to 0 degrees
- moved R8 15.1 mm to (164.3, 93.7)
- moved C8 14.9 mm to (162.1, 109.5), turned to 180 degrees
- moved R2 14.8 mm to (173.9, 135.1), turned to 180 degrees
- moved R9 14.5 mm to (162.1, 106.2), turned to 0 degrees
- moved P1 13.8 mm to (155.7, 96.0)
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Connections:
- net /Amp Potencia/DAC renamed /DAC
- net /Conector/ADC1 renamed /ADC
- C2 pad 2: Net-(C2-Pad2) -> GNDA
- C3 pad 1: Net-(C2-Pad2) -> Net-(C3-Pad1)
- C4 pad 1: Net-(C4-Pad1) -> Net-(C3-Pad2)
- C4 pad 2: GNDA -> Net-(C4-Pad2)
- R1 pad 1: +5V -> +3.3V
- R3 pad 1: Net-(C3-Pad2) -> Net-(C4-Pad2)
- R4 pad 1: GNDA -> Net-(C5-Pad2)
- R4 pad 2: Net-(C2-Pad2) -> Net-(C2-Pad1)
- R5 pad 2: Net-(C3-Pad2) -> Net-(C4-Pad2)
- R6 pad 1: Net-(C5-Pad2) -> GNDA
- R6 pad 2: Net-(C4-Pad1) -> Net-(C3-Pad2)
- RV1 pad 2: Net-(C2-Pad1) -> Net-(C3-Pad1)
- U1 pad 4: GNDA -> GND
- U1 pad 7: +5V -> +3.3V
- U2 pad 4: GNDA -> GND
- XA1 pad 20: Net-(XA1-Pad20) -> GND
- XA1 pad 22: Net-(XA1-Pad22) -> GND
- XA1 pad 24: Net-(XA1-Pad24) -> GND
- XA1 pad 26: Net-(XA1-Pad26) -> GND
- XA1 pad 28: Net-(XA1-Pad28) -> GND
- XA1 pad 30: Net-(XA1-Pad30) -> GND
- XA1 pad 32: Net-(XA1-Pad32) -> GND
- XA1 pad 38: Net-(XA1-Pad38) -> GND
- XA1 pad 4: Net-(XA1-Pad4) -> GND
- XA1 pad 40: Net-(XA1-Pad40) -> GND
Routing:
- net Net-(C3-Pad2): track 57.4 -> 9.63 mm, vias 2 -> 0
- net Net-(C8-Pad1): track 18.2 -> 58.1 mm, vias 2 -> 0
- net GNDA: track 13.8 -> 0.00 mm, vias 4 -> 0
- net Net-(C4-Pad2): track 0.00 -> 12.2 mm
- net Net-(R5-Pad1): track 4.35 -> 13.3 mm, vias 1 -> 0
- net Net-(C4-Pad1): track 7.81 -> 0.00 mm, vias 1 -> 0
- net Net-(RV2-Pad2): track 9.54 -> 16.9 mm, vias 1 -> 0
- net Net-(C5-Pad2): track 17.6 -> 24.6 mm, vias 1 -> 0
- net Net-(C2-Pad2): track 6.82 -> 0.00 mm
- net /ADC: track 15.1 -> 21.3 mm
- net Net-(C3-Pad1): track 0.00 -> 5.25 mm
- net Net-(C5-Pad1): track 23.0 -> 26.4 mm, vias 1 -> 2
- net Net-(C6-Pad2): track 6.48 -> 4.38 mm, vias 1 -> 0
- net +5V: track 1.93 -> 0.00 mm
- net Net-(C1-Pad1): track 13.3 -> 11.4 mm, vias 1 -> 0
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- added copper zone on F.Cu, net +3.3V
- added copper zone on B.Cu, net GND
Other:
- outline, holes or cut-outs redrawn
- net class Default: clearance 0.2 -> 0.3048; trace_width 0.25 -> 0.3048
- rule trace_clearance: 0.2 -> 0.3048
- rule trace_min: 0.2 -> 0.3048
- board text added: "MIC"
- board text added: "SALIDA"

Commit message: v1.3
Routing:
- net GNDA: track 0.00 -> 19.0 mm, vias 0 -> 3
- net GND: track 0.00 -> 2.44 mm, vias 0 -> 1
Changed lines of the file:
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@@
   (general
     (links 60)
-    (no_connects 7)
-    (area 151.689999 73.584999 192.480001 143.585001)
+    (no_connects 1)
+    (area 139.447199 65.659 201.295001 153.670001)
     (thickness 1.6)
     (drawings 6)
-    (tracks 87)
+    (tracks 103)
     (zones 0)
     (modules 31)
@@
   (layers
     (0 F.Cu signal hide)
-    (31 B.Cu signal)
+    (31 B.Cu signal hide)
     (32 B.Adhes user hide)
     (33 F.Adhes user hide)
@@
   (segment (start 175.863 135.128) (end 175.863 139.224) (width 0.3048) (layer F.Cu) (net 1))
   (segment (start 175.863 139.224) (end 175.006 140.081) (width 0.3048) (layer F.Cu) (net 1))
+  (via (at 166.243 107.823) (size 0.6) (drill 0.4) (layers F.Cu B.Cu) (net 2))
+  (segment (start 164.592 106.172) (end 166.243 107.823) (width 0.3048) (layer F.Cu) (net 2))
+  (segment (start 171.863 135.128) (end 171.863 138.938) (width 0.3048) (layer F.Cu) (net 2))
+  (segment (start 171.863 138.938) (end 173.006 140.081) (width 0.3048) (layer F.Cu) (net 2))
+  (segment (start 160.052 123.444) (end 158.115 123.444) (width 0.3048) (layer F.Cu) (net 2))
+  (segment (start 156.591 124.968) (end 156.21 124.968) (width 0.3048) (layer F.Cu) (net 2))
+  (segment (start 158.115 123.444) (end 156.591 124.968) (width 0.3048) (layer F.Cu) (net 2))
+  (segment (start 156.21 124.968) (end 155.956 125.222) (width 0.3048) (layer F.Cu) (net 2))
+  (segment (start 179.959 132.683) (end 179.959 135.001) (width 0.3048) (layer F.Cu) (net 2))
+  (via (at 179.959 135.001) (size 0.6) (drill 0.4) (layers F.Cu B.Cu) (net 2))
+  (segment (start 164.052 106.172) (end 164.592 106.172) (width 0.3048) (layer F.Cu) (net 2))
+  (segment (start 164.052 116.332) (end 165.227 116.332) (width 0.3048) (layer F.Cu) (net 2))
+  (via (at 166.878 117.983) (size 0.6) (drill 0.4) (layers F.Cu B.Cu) (net 2))
+  (segment (start 165.227 116.332) (end 166.878 117.983) (width 0.3048) (layer F.Cu) (net 2))
   (segment (start 160.052 116.332) (end 160.052 112.776) (width 0.3048) (layer F.Cu) (net 3))
   (segment (start 161.036 128.27) (end 161.036 126.873) (width 0.3048) (layer F.Cu) (net 4))
@@
   (segment (start 167.767 103.505) (end 169.164 102.108) (width 0.3048) (layer F.Cu) (net 45))
   (segment (start 157.861 103.505) (end 167.767 103.505) (width 0.3048) (layer F.Cu) (net 45))
+  (segment (start 179.959 128.683) (end 179.959 126.238) (width 0.3048) (layer F.Cu) (net 46))
+  (via (at 179.959 126.238) (size 0.6) (drill 0.4) (layers F.Cu B.Cu) (net 46))
   (zone (net 2) (net_name GNDA) (layer B.Cu) (hatch edge 0.508)
     (connect_pads (clearance 0.508))
