File: buttons.sch (KiCad schematic (older format))
At the start: 16 parts, among them SW1 SW_PUSH, SW2 SW_PUSH, SW3 SW_PUSH, SW4 SW_PUSH, SW5 SW_PUSH, SW6 SW_PUSH, SW7 SW_PUSH, SW8 SW_PUSH

Commit message: Finaliza proyecto en ultima clase de diseno PCB. Ultimos cambios en el repo.
Parts:
- R1, R2: Digikey# 680EBK­ND -> 680EBK-ND
- R3, R4, R5, R6, R7, R8: footprint footprints:Resistor_Horizontal_RM7mm -> simonShield:Resistor_Horizontal_RM7mm; Digikey# 680EBK­ND -> 680EBK-ND
- SW1, SW2, SW3, SW4, SW5, SW6, SW7, SW8: footprint footprints:SW_PUSH_SMALL -> simonShield:SW_PUSH_SMALL; Digikey# 450­1804­ND -> 450-1804-ND
Connections:
- net labels added: VCC
- net labels removed: VDD
