File: TP.kicad_pcb (KiCad board)
At the start: 2 copper layers, 42 x 61 mm, 18 parts, among them J1 DB9, U1 AFE4490, Y1 8MHz

Commit message: Version con correcciones
Parts:
- added Fid: Fiducial_1mm_Dia_2.54mm_Outer_CopperTop, Fiducials:Fiducial_1mm_Dia_2.54mm_Outer_CopperTop, F.Cu at (181.4, 100.6)
- Oximentro : renamed from G***
- moved Oximentro  0.46 mm to (163.6, 149.3)
Routing:
- net +3V3: track 115.2 -> 113.1 mm
- net Net-(J1-Pad2): track 43.2 -> 44.8 mm
- net Net-(U1-Pad20): track 80.8 -> 79.7 mm
- net GND: track 144.7 -> 145.7 mm
- net Net-(U1-Pad21): track 75.3 -> 74.2 mm
- net Net-(U1-Pad28): track 50.4 -> 49.8 mm
- added copper zone on F.Cu, net +3V3
- added copper zone on F.Cu, net GND
Other:
- net class Default: clearance 0.2 -> 0.24
- rule trace_clearance: 0.2 -> 0.24
- rule trace_min: 0.2 -> 0.1
- board text added: "Ancho minimo de pista 0,25 mm Diametro agujero via 0,50 mm Diametro de via 1,00 mm"
- board text added: "Diseño doble faz. Sin requerimientos especiales."
- board text added: "Fernando Meira Curso PCB - CESE"
- board text added: "Grilla de posicionamiento: 0,50 mm"
- board text added: "Grilla de ruteo: 0,10 mm"
- board text added: "Industria Argentina"
- board text added: "STACK-UP"

Commit message: Version con correcciones
Parts:
- Oximetro : renamed from Oximentro 
- moved Oximetro  40.9 mm to (143.2, 113.8)
- moved Fid 31.8 mm to (161.2, 76.1)
- moved R2 31.8 mm to (141.6, 89.2)
- moved XA1 31.8 mm to (127.8, 79.5)
- moved C1 31.8 mm to (150.8, 93.0)
- moved C10 31.8 mm to (157.3, 78.5)
- moved C11 31.8 mm to (147.3, 78.5)
- moved C2 31.8 mm to (155.3, 93.0)
- moved C3 31.8 mm to (146.3, 97.5)
- moved C4 31.8 mm to (146.3, 93.0)
- moved C5 31.8 mm to (150.8, 97.5)
- moved C6 31.8 mm to (155.3, 97.5)
- moved C7 31.8 mm to (159.1, 88.8)
- moved C8 31.8 mm to (159.1, 83.2)
- moved C9 31.8 mm to (152.3, 78.5)
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Routing:
- net Net-(U1-Pad26): track 38.3 -> 42.2 mm
- net GND: track 145.7 -> 141.9 mm
- net Net-(U1-Pad27): track 49.7 -> 48.2 mm
- net Net-(U1-Pad25): track 33.9 -> 32.4 mm
- net Net-(J1-Pad3): track 46.2 -> 47.1 mm
- net Net-(C2-Pad1): track 12.8 -> 12.1 mm
Other:
- board size 42 x 61 mm -> 41.9 x 61 mm
- rule trace_min: 0.1 -> 0.24
