File: modelos/Basico/basico.kicad_pcb (KiCad board)
At the start: 2 copper layers, 85.7 x 60.3 mm, 5 parts

Commit message: Detalles NC y power flag en .sch. Lock conector y anchos pista en PCB.
Other:
- net class Default: clearance 0.508 -> 0.51
- rule trace_clearance: 0.508 -> 0.51
Changed lines of the file:
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@@
     (links 28)
     (no_connects 28)
-    (area 59.614999 80.569999 145.490001 141.045001)
+    (area 17.422141 15.774999 279.500001 163.930001)
     (thickness 1.6)
     (drawings 35)
@@
     (last_trace_width 0.381)
     (user_trace_width 0.508)
-    (user_trace_width 0.635)
-    (user_trace_width 0.762)
+    (user_trace_width 0.6)
+    (user_trace_width 0.6)
+    (user_trace_width 0.8)
+    (user_trace_width 1)
     (user_trace_width 1.016)
     (user_trace_width 1.27)
-    (user_trace_width 1.524)
-    (trace_clearance 0.508)
+    (user_trace_width 2)
+    (trace_clearance 0.51)
     (zone_clearance 0.508)
     (zone_45_only no)
@@
   (net 4 GNDA)
   (net_class Default "This is the default net class."
-    (clearance 0.508)
+    (clearance 0.51)
     (trace_width 0.381)
     (via_dia 0.6)
@@
     (add_net GNDA)
   )
-  (module footprint:Conn_Poncho_SinBorde (layer F.Cu)
+  (module footprint:Conn_Poncho_SinBorde locked (layer F.Cu)
     (at 137.16 86.36)
     (tags "CONN Poncho")
