File: Pico_WiFi/DISEÑO_PONCHO_WIFI_PICOCIAA.sch (KiCad schematic (older format))
At the start: 11 parts, among them P1 MOUNT_HOLE, P2 MOUNT_HOLE, U1 ESP-12E

Commit message: Actualizo Poncho pico-wifi desde https://github.com/sergiordj/Poncho_wifi_picociaa
Parts:
- removed R4, R5: R, Resistors_SMD:R_0805_HandSoldering, symbol R
- added FID1, FID2, FID3: FIDUCIAL, Poncho_wifi:Fiducial_1mm_Dia_2.54mm_Outer_CopperTop, symbol FIDUCIAL
- Conn1: footprint pico_ciaa_ponchos:Conn_Pico_Ciaa -> Poncho_wifi:Conn_Pico_Ciaa
- P1, P2: footprint footprints:PIN_ARRAY_1 -> Poncho_wifi:PIN_ARRAY_1
- R1, R2, R3, R6, R7: footprint Resistors_SMD:R_0805_HandSoldering -> Poncho_wifi:R_0805_HandSoldering; Digikey# (none) -> 1056-MCR10J103-CHP
- U1: footprint pico_ciaa_ponchos:ESP-12E -> Poncho_wifi:ESP-12E; Digikey# (none) -> 1528-1438-ND
Connections:
- wire segments 52 -> 51
- no-connect marks 32 -> 25
Other:
- moved on the sheet: R3
